File: acondicionador/acondicionador.kicad_sch (KiCad schematic)
At the start: 35 parts, among them J1 VC_24V, J2 Ant, J4 SMA, U1 TL084, U2 TL082, U3 LM7818_TO220, U4 AD620

Commit message: Modificación posición C5 C6 en placa Acondicionador y cambio de huella sma (verificar), cambio de huella sma en placa Adquisición (verificar)
Parts:
- J4: footprint Connector_Coaxial:SMA_Amphenol_132289_EdgeMount -> Connector_Coaxial:SMA_Samtec_SMA-J-P-H-ST-EM1_EdgeMount
Changed lines of the file:
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@@
 	)
 	(junction
+		(at 34.29 52.07)
+		(diameter 0)
+		(color 0 0 0 0)
+	)
+	(junction
 		(at 91.44 139.7)
 		(diameter 0)
@@
 	)
 	(junction
+		(at 34.29 36.83)
+		(diameter 0)
+		(color 0 0 0 0)
+	)
+	(junction
 		(at 96.52 52.07)
 		(diameter 0)
@@
 	)
 	(junction
-		(at 58.42 36.83)
+		(at 91.44 95.25)
 		(diameter 0)
 		(color 0 0 0 0)
 	)
 	(junction
-		(at 91.44 95.25)
+		(at 58.42 36.83)
 		(diameter 0)
 		(color 0 0 0 0)
@@
 	(wire
 		(pts
-			(xy 58.42 36.83) (xy 71.12 36.83)
-		)
-		(stroke
-			(width 0)
-			(type default)
-		)
-	)
-	(wire
-		(pts
 			(xy 34.29 52.07) (xy 46.99 52.07)
 		)
@@
 	(wire
 		(pts
+			(xy 58.42 36.83) (xy 71.12 36.83)
+		)
+		(stroke
+			(width 0)
+			(type default)
+		)
+	)
+	(wire
+		(pts
 			(xy 78.74 52.07) (xy 96.52 52.07)
 		)
@@
 	)
 	(symbol
+		(lib_id "power:PWR_FLAG")
+		(at 34.29 36.83 0)
+		(unit 1)
+		(exclude_from_sim no)
+		(in_bom yes)
+		(on_board yes)
+		(dnp no)
+		(fields_autoplaced yes)
+		(property "Reference" "#FLG01"
+			(at 34.29 34.925 0)
+			(effects
+				(font
+					(size 1.27 1.27)
+				)
+				(hide yes)
+			)
+		)
+		(property "Value" "PWR_FLAG"
+			(at 34.29 31.75 0)
+			(effects
+				(font
+					(size 1.27 1.27)
+				)
+			)
+		)
+		(property "Footprint" ""
+			(at 34.29 36.83 0)
+			(effects
+				(font
+					(size 1.27 1.27)
+				)
+				(hide yes)
+			)
+		)
+		(property "Datasheet" "~"
+			(at 34.29 36.83 0)
+			(effects
+				(font
+					(size 1.27 1.27)
+				)
+				(hide yes)
+			)
+		)
+		(property "Description" "Special symbol for telling ERC where power comes from"
+			(at 34.29 36.83 0)
+			(effects
+				(font
+					(size 1.27 1.27)
+				)
+				(hide yes)
+			)
+		)
+		(pin "1"
+		)
+		(instances
+			(project ""
+				(path "/d06a90f2-131c-4d35-8833-41ab8319c85a"
+					(reference "#FLG01")
+					(unit 1)
+				)
+			)
+		)
+	)
+	(symbol
 		(lib_id "power:GND")
 		(at 203.2 142.24 0)
@@
 	)
 	(symbol
+		(lib_id "power:PWR_FLAG")
+		(at 34.29 52.07 180)
+		(unit 1)
+		(exclude_from_sim no)
+		(in_bom yes)
+		(on_board yes)
+		(dnp no)
+		(property "Reference" "#FLG02"
+			(at 34.29 53.975 0)
+			(effects
+				(font
+					(size 1.27 1.27)
+				)
+				(hide yes)
+			)
+		)
+		(property "Value" "PWR_FLAG"
+			(at 34.29 56.134 0)
+			(effects
+				(font
+					(size 1.27 1.27)
+				)
+			)
+		)
+		(property "Footprint" ""
+			(at 34.29 52.07 0)
+			(effects
+				(font
+					(size 1.27 1.27)
+				)
+				(hide yes)
+			)
+		)
+		(property "Datasheet" "~"
+			(at 34.29 52.07 0)
+			(effects
+				(font
+					(size 1.27 1.27)
+				)
+				(hide yes)
+			)
+		)
+		(property "Description" "Special symbol for telling ERC where power comes from"
+			(at 34.29 52.07 0)
+			(effects
+				(font
+					(size 1.27 1.27)
+				)
+				(hide yes)
+			)
+		)
+		(pin "1"
+		)
+		(instances
+			(project "acondicionador"
+				(path "/d06a90f2-131c-4d35-8833-41ab8319c85a"
+					(reference "#FLG02")
+					(unit 1)
+				)
+			)
+		)
+	)
+	(symbol
 		(lib_id "Device:C_Polarized_US")
 		(at 46.99 43.18 0)
@@
 			)
 		)
-		(property "Footprint" "Connector_Coaxial:SMA_Amphenol_132289_EdgeMount"
+		(property "Footprint" "Connector_Coaxial:SMA_Samtec_SMA-J-P-H-ST-EM1_EdgeMount"
 			(at 247.65 111.76 0)
 			(effects

Commit message: Compensación Voi acondicionador
Parts:
- added R15: 750k, huellas_proyecto:R_Axial_DIN0207_L6.3mm_D2.5mm_P10.16mm_Horizontal-pad2mm, symbol Device:R_US
- added RV2: 10k, huellas_proyecto:Potentiometer_Bourns_3296W_Vertical-pad2mm, symbol Device:R_Potentiometer_Trim_US
Connections:
- net GND: now also RV2.3
- net VCC: now also RV2.1
- net at R3.1, U1.12 (+): now also R15.1
- new net: R15.2, RV2.2
Other:
- note added: "Comp. Vio"
